File: Windturbine.sch (EAGLE design)
At the start: 14 parts, among them IC1 LM2576S, U1 328P

Commit message: Add files via upload
Parts:
- removed B1: (no value), pololu:POLOLU_1183
- removed U$1: RESISTOR, tango:RESISTOR
- added A988: (no value), pololu:POLOLU_1183
- added C3: 100u, resistor:C-US050-045X075
- U1: value 328P -> Atmega328p
- renumbered S1 to CONTROL, U$2 to +12V, U$3 to FOR_ON_OFF_SIGNAL
Connections:
- new net +5V: A988.VDD, U1.VCC
- new net N$11: A988.GND_SUPP, C3.2
- new net TO_STEPPER_MOTOR(BLK): A988.2B
- new net TO_STEPPER_MOTOR(BLU): A988.1B
- new net TO_STEPPER_MOTOR(GRN): A988.2A
- new net TO_STEPPER_MOTOR(RED): A988.1A
- net N$1: now also A988.DIR, U1.PD4(XCK/T0); no longer B1.!RESET, B1.!SLEEP
- net N$2: now also A988.V_MOT, C3.1; no longer B1.DIR, U1.PD4(XCK/T0)
- net N$3: now also A988.STEP; no longer B1.STEP
- net N$4: now also A988.!ENABLE; no longer B1.!ENABLE
- net PE: now also A988.GND1, U1.GND
Other:
- moved on the sheet: U1, X1

Commit message: Add files via upload
Parts:
- added ANEMOMETER, WIND_VANE: -CON3, tango:-CON3
- added MOTOR_SUPPLY: 12V, battery:3V11R
- added U$1: LCD-HD447803-HOLES16X2-3-HOLES, HD44780LCD:LCD-HD447803-HOLES16X2-3-HOLES
Connections:
- removed net +5V: A988.VDD, U1.VCC
- removed net PE: +12V.2, A988.GND1, C1.2, C2.2, CONTROL.S, D1.A, FOR_ON_OFF_SIGNAL.1, IC1.GND, LED1.CATHODE, U1.GND, X1.4
- new net INT_SIGNAL: ANEMOMETER.2, U1.PD2(INT0)
- new net N$12: U$1.RS, U1.PB0(ICP)
- new net N$13: U$1.E, U1.PB1(OC1A)
- new net N$14: U$1.DB4, U1.PB4(MISO)
- new net N$15: U$1.DB5, U1.PB5(SCK)
- new net N$16: U$1.DB6, U1.PB6(XTAL1/TOSC1)
- new net N$17: U$1.DB7, U1.PB7(XTAL2/TOSC2)
- new net NEG: +12V.2, A988.GND1, ANEMOMETER.1, C1.2, C2.2, CONTROL.S, D1.A, FOR_ON_OFF_SIGNAL.1, IC1.GND, LED1.CATHODE, U$1.R/W, U1.GND, WIND_VANE.1, X1.4
- new net POS: A988.VDD, ANEMOMETER.3, U$1.VDD, U1.VCC, WIND_VANE.3
- new net SIGNAL: U1.PC0(ADC0), WIND_VANE.2
- net N$11: now also MOTOR_SUPPLY.-
- net N$2: now also MOTOR_SUPPLY.+
Other:
- moved on the sheet: A988
