File: Windturbine1.sch (EAGLE design)
At the start: 19 parts, among them IC1 LM2576S, U1 Atmega328p

Commit message: Add files via upload
Parts:
- added JP1: (no value), arduino_jw:ARDUINO_CONN-ICSP
Connections:
- removed net N$15: U$1.DB5, U1.PB5(SCK)
- new net +5V: JP1.2
- new net GND: JP1.6
- new net N$20: JP1.3, U$1.DB5, U1.PB5(SCK)
- new net N$21: JP1.5
- net N$14: now also JP1.1, JP1.4, U1.PB3(MOSI/OC2)
Changed lines of the file:
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@@
 <?xml version="1.0" encoding="utf-8"?>
 <!DOCTYPE eagle SYSTEM "eagle.dtd">
-<eagle version="9.2.1">
+<eagle version="9.1.3">
 <drawing>
 <settings>
@@
 <part name="U$1" library="HD44780LCD" deviceset="LCD-HD44780" device="16X2-3-HOLES" technology="3-HOLES"/>
 <part name="ANEMOMETER" library="tango" deviceset="-CON3" device=""/>
-<part name="C4" library="docu-dummy" library_urn="urn:adsk.eagle:library:215" deviceset="C" device=""/>
-<part name="C5" library="docu-dummy" library_urn="urn:adsk.eagle:library:215" deviceset="C" device=""/>
+<part name="C4" library="docu-dummy" library_urn="urn:adsk.eagle:library:215" deviceset="C" device="" value="22pF"/>
+<part name="C5" library="docu-dummy" library_urn="urn:adsk.eagle:library:215" deviceset="C" device="" value="22pF"/>
 <part name="X_1" library="ngspice-simulation" library_urn="urn:adsk.eagle:library:527439" deviceset="GND" device=""/>
 <part name="U$2" library="crystal" deviceset="90SMX" device=""/>
 <part name="X_2" library="ngspice-simulation" library_urn="urn:adsk.eagle:library:527439" deviceset="GND" device=""/>
+<part name="JP1" library="arduino_jw" deviceset="ARDUINO_CONN-ICSP" device=""/>
+<part name="P+2" library="supply1" library_urn="urn:adsk.eagle:library:371" deviceset="+5V" device=""/>
+<part name="GND1" library="supply1" library_urn="urn:adsk.eagle:library:371" deviceset="GND" device=""/>
 </parts>
 <sheets>
@@
 <instance part="C5" gate="G$1" x="86.36" y="-15.24" smashed="yes"/>
 <instance part="X_1" gate="G$1" x="76.2" y="-22.86" smashed="yes"/>
-<instance part="U$2" gate="G$1" x="81.28" y="-12.7" smashed="yes">
-<attribute name="NAME" x="78.74" y="-10.414" size="1.778" layer="95"/>
-<attribute name="VALUE" x="78.74" y="-16.51" size="1.778" layer="96"/>
-</instance>
+<instance part="U$2" gate="G$1" x="81.28" y="-12.7" smashed="yes"/>
 <instance part="X_2" gate="G$1" x="86.36" y="-22.86" smashed="yes"/>
+<instance part="JP1" gate="G$1" x="114.3" y="-40.64"/>
+<instance part="P+2" gate="1" x="139.7" y="-20.32" smashed="yes">
+<attribute name="VALUE" x="142.24" y="-17.78" size="1.778" layer="96" rot="R180"/>
+</instance>
+<instance part="GND1" gate="1" x="139.7" y="-45.72"/>
 </instances>
 <busses>
@@
 <wire x1="152.4" y1="78.74" x2="152.4" y2="50.8" width="0.1524" layer="91"/>
 <wire x1="152.4" y1="50.8" x2="132.08" y2="30.48" width="0.1524" layer="91"/>
-<wire x1="132.08" y1="30.48" x2="132.08" y2="10.16" width="0.1524" layer="91"/>
+<wire x1="132.08" y1="30.48" x2="132.08" y2="12.7" width="0.1524" layer="91"/>
 <pinref part="U1" gate="U1" pin="PB4(MISO)"/>
+<wire x1="132.08" y1="12.7" x2="132.08" y2="10.16" width="0.1524" layer="91"/>
 <wire x1="132.08" y1="10.16" x2="129.54" y2="10.16" width="0.1524" layer="91"/>
-</segment>
-</net>
-<net name="N$15" class="0">
-<segment>
-<pinref part="U$1" gate="G$1" pin="DB5"/>
-<wire x1="160.02" y1="76.2" x2="149.86" y2="76.2" width="0.1524" layer="91"/>
-<wire x1="149.86" y1="76.2" x2="149.86" y2="50.8" width="0.1524" layer="91"/>
-<wire x1="149.86" y1="50.8" x2="139.7" y2="40.64" width="0.1524" layer="91"/>
-<wire x1="139.7" y1="40.64" x2="139.7" y2="30.48" width="0.1524" layer="91"/>
-<wire x1="139.7" y1="30.48" x2="139.7" y2="15.24" width="0.1524" layer="91"/>
-<wire x1="139.7" y1="15.24" x2="132.08" y2="7.62" width="0.1524" layer="91"/>
-<pinref part="U1" gate="U1" pin="PB5(SCK)"/>
-<wire x1="132.08" y1="7.62" x2="129.54" y2="7.62" width="0.1524" layer="91"/>
+<pinref part="JP1" gate="G$1" pin="1"/>
+<wire x1="129.54" y1="-25.4" x2="132.08" y2="-25.4" width="0.1524" layer="91"/>
+<wire x1="132.08" y1="-25.4" x2="132.08" y2="10.16" width="0.1524" layer="91"/>
+<wire x1="132.08" y1="10.16" x2="129.54" y2="10.16" width="0.1524" layer="91"/>
+<junction x="129.54" y="10.16"/>
+<pinref part="JP1" gate="G$1" pin="4"/>
+<wire x1="129.54" y1="-33.02" x2="137.16" y2="-33.02" width="0.1524" layer="91"/>
+<wire x1="137.16" y1="-33.02" x2="137.16" y2="5.08" width="0.1524" layer="91"/>
+<pinref part="U1" gate="U1" pin="PB3(MOSI/OC2)"/>
+<wire x1="137.16" y1="5.08" x2="137.16" y2="12.7" width="0.1524" layer="91"/>
+<wire x1="137.16" y1="12.7" x2="132.08" y2="12.7" width="0.1524" layer="91"/>
+<junction x="132.08" y="12.7"/>
+<wire x1="132.08" y1="12.7" x2="129.54" y2="12.7" width="0.1524" layer="91"/>
 </segment>
 </net>
@@
 </segment>
 </net>
+<net name="+5V" class="0">
+<segment>
+<pinref part="JP1" gate="G$1" pin="2"/>
+<wire x1="129.54" y1="-27.94" x2="139.7" y2="-27.94" width="0.1524" layer="91"/>
+<wire x1="139.7" y1="-27.94" x2="139.7" y2="-22.86" width="0.1524" layer="91"/>
+<pinref part="P+2" gate="1" pin="+5V"/>
+</segment>
+</net>
+<net name="GND" class="0">
+<segment>
+<pinref part="JP1" gate="G$1" pin="6"/>
+<wire x1="129.54" y1="-38.1" x2="139.7" y2="-38.1" width="0.1524" layer="91"/>
+<wire x1="139.7" y1="-38.1" x2="139.7" y2="-43.18" width="0.1524" layer="91"/>
+<pinref part="GND1" gate="1" pin="GND"/>
+</segment>
+</net>
+<net name="N$20" class="0">
+<segment>
+<pinref part="JP1" gate="G$1" pin="3"/>
+<wire x1="129.54" y1="-30.48" x2="134.62" y2="-30.48" width="0.1524" layer="91"/>
+<wire x1="134.62" y1="-30.48" x2="134.62" y2="5.08" width="0.1524" layer="91"/>
+<wire x1="134.62" y1="5.08" x2="129.54" y2="5.08" width="0.1524" layer="91"/>
+<pinref part="U$1" gate="G$1" pin="DB5"/>
+<wire x1="160.02" y1="76.2" x2="149.86" y2="76.2" width="0.1524" layer="91"/>
+<wire x1="149.86" y1="76.2" x2="149.86" y2="50.8" width="0.1524" layer="91"/>
+<wire x1="149.86" y1="50.8" x2="139.7" y2="40.64" width="0.1524" layer="91"/>
+<wire x1="139.7" y1="40.64" x2="139.7" y2="30.48" width="0.1524" layer="91"/>
+<wire x1="139.7" y1="30.48" x2="139.7" y2="15.24" width="0.1524" layer="91"/>
+<wire x1="139.7" y1="15.24" x2="132.08" y2="7.62" width="0.1524" layer="91"/>
+<pinref part="U1" gate="U1" pin="PB5(SCK)"/>
+<wire x1="132.08" y1="7.62" x2="129.54" y2="7.62" width="0.1524" layer="91"/>
+<wire x1="129.54" y1="5.08" x2="129.54" y2="7.62" width="0.1524" layer="91"/>
+<junction x="129.54" y="7.62"/>
+</segment>
+</net>
+<net name="N$21" class="0">
+<segment>
+<pinref part="JP1" gate="G$1" pin="5"/>
+<wire x1="129.54" y1="-35.56" x2="160.02" y2="-35.56" width="0.1524" layer="91"/>
+<wire x1="160.02" y1="-35.56" x2="160.02" y2="-40.64" width="0.1524" layer="91"/>
+</segment>
+</net>
