File: Voltage2.sch (EAGLE design)
At the start: 11 parts, among them IC1 317T, IC2 ACS712-LC, Q1 FDN340P, U1 TEXAS_INSTRUMENTS_LMV358IDGKR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, U2 LP2985-33DBVR, U3 TEXAS_INSTRUMENTS_LMV358IDGKR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, U4 NCP1117ST50T3G

Commit message: Add files via upload
Parts:
- added C1: 1nF, SparkFun-Capacitors:1.0NF/1000PF-0603-50V-10%
- added C2, C7: 47uF, SparkFun-Capacitors:47UF-POLAR-EIA3528-10V-10%
- added C4: 1.0uF, SparkFun-Capacitors:1.0UF-0603-16V-10%
- added C5, C6: 100nF, resistor:C-USC0603
- added D5: 1N5060GP, diode:1N5060GP
- added R1, R2, R8, R9: 1k, SparkFun-Resistors:1KOHM-0603-1/10W-1%
- added R10, R3: 10k, SparkFun-Resistors:10KOHM-0603-1/10W-1%
- added R4: ERJ-3EKF2152V, ERJ-3EKF2152V:ERJ-3EKF2152V
- added R5: ERJ-3EKF1131V, ERJ-3EKF1131V:ERJ-3EKF1131V
Connections:
- new net 10K: R10.2
- new net 47U: C2.-
- new net VIN: R4.2
- new net VOUT: R4.1, R5.2
- net +3V3: now also C4.1
- net +5V: now also C5.2, R1.1, R2.1, R9.1
- net 100N: now also C6.1, C7.+
- net 1K: now also R8.2
- net CMP: now also R10.1, R3.2
- net GND: now also C1.2, C4.2, C5.1, C6.2, C7.-, R3.1, R5.1
- net N$1: now also R1.2, R2.2
- net N$11: now also C2.+, D5.C
- net N$12: now also C1.1
- net N$3: now also D5.A
- net N$7: now also R9.2
- net N$9: now also R8.1
